Commit message: Mirror ORCA left URDF properly + mirrored meshes
The previous orca_left_6dof.urdf was a copy of the right URDF with
right_-/L_- token rename only, so the left hand carried right-handed
finger geometry. dex_retargeting compensated by rotating the wrist
~pi around yaw, producing the visible '180 degrees around the wrist'
artefact and a 3.6x higher left-vs-right control error (0.26 vs 0.07).

Generate a properly mirrored left URDF from the right via
hand_proc/mirror_orca_urdf.py:
- Reflect every <origin xyz=".."/> on x and <origin rpy="..."/> on
  pitch/yaw (YZ-plane mirror, validated against the geort bundle's
  hand-built mirror at orca_v1b_left/orcahand_left.urdf).
- Keep <axis xyz="..."/> unchanged — dex_retargeting's SLSQP only
  cares about fingertip-vector distance, so it finds the right qpos
  whichever sign represents 'flexion'. Negating axes additionally
  would invert the joint-limit semantics and broke retargeting
  empirically (left err: 0.13 with origins-only flip, 2.57 with full
  axis negation).
- Repoint mesh refs at left_meshes/, populated with the already
  mirrored visual + collision STLs from real2sim2target's GeoRT
  bundle (md5 != right; truly reflected geometry).

Post-fix retargeting on box-0-600: left control err 0.13 (was 0.26),
right unchanged at 0.05. Wrist no longer rotates ~pi to compensate.

File: dexmachina/assets/orca_hand/orca_left_6dof.urdf (robot description, URDF)
Before this commit: robot orcahand_v1b_left_6dof, 45 links, 44 joints
Links:
- link left_index_ip: geometry collision mesh filename=left_meshes/converted_index_ip_mesh.stl; visual mesh filename=left_meshes/converted_index_ip_mesh.stl
- link left_index_mp: geometry collision mesh filename=left_meshes/converted_index_mp_mesh.stl; visual mesh filename=left_meshes/converted_index_mp_mesh.stl
- link left_index_pp: geometry collision mesh filename=left_meshes/converted_index_pp_mesh.stl; visual mesh filename=left_meshes/converted_index_pp_mesh.stl
- link left_middle_ip: geometry collision mesh filename=left_meshes/converted_middle_ip_mesh.stl; visual mesh filename=left_meshes/converted_middle_ip_mesh.stl
- link left_middle_mp: geometry collision mesh filename=left_meshes/converted_middle_mp_mesh.stl; visual mesh filename=left_meshes/converted_middle_mp_mesh.stl
- link left_middle_pp: geometry collision mesh filename=left_meshes/converted_middle_pp_mesh.stl; visual mesh filename=left_meshes/converted_middle_pp_mesh.stl
- link left_palm: geometry collision mesh filename=left_meshes/converted_palm_mesh.stl; visual mesh filename=left_meshes/converted_palm_mesh.stl
- link left_pinky_ip: geometry collision mesh filename=left_meshes/converted_pinky_ip_mesh.stl; visual mesh filename=left_meshes/converted_pinky_ip_mesh.stl
- link left_pinky_mp: geometry collision mesh filename=left_meshes/converted_pinky_mp_mesh.stl; visual mesh filename=left_meshes/converted_pinky_mp_mesh.stl
- link left_pinky_pp: geometry collision mesh filename=left_meshes/converted_pinky_pp_mesh.stl; visual mesh filename=left_meshes/converted_pinky_pp_mesh.stl
- link left_ring_ip: geometry collision mesh filename=left_meshes/converted_ring_ip_mesh.stl; visual mesh filename=left_meshes/converted_ring_ip_mesh.stl
- link left_ring_mp: geometry collision mesh filename=left_meshes/converted_ring_mp_mesh.stl; visual mesh filename=left_meshes/converted_ring_mp_mesh.stl
- link left_ring_pp: geometry collision mesh filename=left_meshes/converted_ring_pp_mesh.stl; visual mesh filename=left_meshes/converted_ring_pp_mesh.stl
- link left_thumb_dp: geometry collision mesh filename=left_meshes/converted_thumb_dp_mesh.stl; visual mesh filename=left_meshes/converted_thumb_dp_mesh.stl
- link left_thumb_ip: geometry collision mesh filename=left_meshes/converted_thumb_ip_mesh.stl; visual mesh filename=left_meshes/converted_thumb_ip_mesh.stl
- link left_thumb_mp: geometry collision mesh filename=left_meshes/converted_thumb_mp_mesh.stl; visual mesh filename=left_meshes/converted_thumb_mp_mesh.stl
- link left_thumb_pp: geometry collision mesh filename=left_meshes/converted_thumb_pp_mesh.stl; visual mesh filename=left_meshes/converted_thumb_pp_mesh.stl
Joints:
- joint L_forearm_wrist_offset: origin xyz=-0.0019999999999999844 0.0014412498723577962 0.038719313535195574 rpy=0.0 0.0 0.0 -> xyz=0.00199999999999998443 0.0014412498723577962 0.038719313535195574 rpy=0.0 0 0
- joint index_ip2index_fingertip_fixed: origin xyz=-0.009 0.0 0.04 rpy=0.0 0.0 0.0 -> xyz=0.00899999999999999932 0.0 0.04 rpy=0.0 0 0
- joint joint_abd_index: origin xyz=-0.024091784930027955 0.0019042822195537508 0.025160679302659018 rpy=1.6066965884733262 1.1355216005349669 -0.053392057607510646 -> xyz=0.0240917849300279555 0.0019042822195537508 0.025160679302659018 rpy=1.6066965884733262 -1.13552160053496687 0.0533920576075106457
- joint joint_abd_index_offset: origin xyz=-0.01999999999999969 -1.222980050563649e-16 -2.6020852139652106e-18 rpy=0.0 0.0 0.0 -> xyz=0.0199999999999996916 -1.222980050563649e-16 -2.6020852139652106e-18 rpy=0.0 0 0
- joint joint_abd_middle: origin xyz=-3.178399083063177e-17 1.2056328158038776e-17 0.02999999999999983 rpy=1.570796326794897 1.5707963267948961 0.0 -> xyz=3.17839908306317727e-17 1.2056328158038776e-17 0.02999999999999983 rpy=1.570796326794897 -1.57079632679489611 0
- joint joint_abd_middle_offset: origin xyz=-0.019999999999999882 4.336808689942018e-18 -9.540979117872439e-18 rpy=0.0 0.0 0.0 -> xyz=0.0199999999999998825 4.336808689942018e-18 -9.540979117872439e-18 rpy=0.0 0 0
- joint joint_abd_pinky: origin xyz=0.042587682827929796 0.004991925321003609 0.007247738795820422 rpy=-1.4969430651841686 0.8614853700810632 -2.8837300965971076 -> xyz=-0.0425876828279297959 0.004991925321003609 0.007247738795820422 rpy=-1.4969430651841686 -0.861485370081063184 2.88373009659710755
- joint joint_abd_pinky_offset: origin xyz=-0.02000000000000019 2.47198095326695e-17 6.158268339717665e-17 rpy=0.0 0.0 0.0 -> xyz=0.0200000000000001912 2.47198095326695e-17 6.158268339717665e-17 rpy=0.0 0 0
- joint joint_abd_ring: origin xyz=0.02151626244325176 0.0015399660708893441 0.020821937215657737 rpy=-1.5359724334240132 1.3083608795701238 -3.0544118070011477 -> xyz=-0.0215162624432517595 0.0015399660708893441 0.020821937215657737 rpy=-1.5359724334240132 -1.30836087957012381 3.05441180700114767
- joint joint_abd_ring_offset: origin xyz=-0.019999999999999712 8.239936510889834e-17 -6.071532165918825e-18 rpy=0.0 0.0 0.0 -> xyz=0.0199999999999997125 8.239936510889834e-17 -6.071532165918825e-18 rpy=0.0 0 0
- joint joint_abd_thumb: origin xyz=-0.028209038238965978 0.01777053753934476 -0.013209503444777428 rpy=0.5385748168211226 -0.05594923693864806 -1.2704659007702708 -> xyz=0.0282090382389659777 0.01777053753934476 -0.013209503444777428 rpy=0.5385748168211226 0.0559492369386480615 1.27046590077027077
- joint joint_abd_thumb_offset: origin xyz=-0.0 -0.0 -0.0 rpy=0.0 0.0 0.0 -> xyz=0 -0.0 -0.0 rpy=0.0 0 0
- joint joint_dip_thumb: origin xyz=0.0004999999999720094 -6.765421556309548e-16 0.03299999999999984 rpy=2.4424906541753483e-15 2.220446049250313e-15 1.4988010832439653e-15 -> xyz=-0.00049999999997200938 -6.765421556309548e-16 0.03299999999999984 rpy=2.4424906541753483e-15 -2.22044604925031308e-15 -1.49880108324396527e-15
- joint joint_dip_thumb_offset: origin xyz=-0.0 -0.0 -0.0 rpy=0.0 0.0 0.0 -> xyz=0 -0.0 -0.0 rpy=0.0 0 0
- joint joint_iip_index: origin xyz=0.0004999999999839698 5.698990924330967e-17 0.03799999999999997 rpy=0.0 0.0 -1.1102230246251565e-16 -> xyz=-0.000499999999983969756 5.698990924330967e-17 0.03799999999999997 rpy=0.0 0 1.11022302462515654e-16
- joint joint_iip_index_offset: origin xyz=5.782630065573341e-18 -2.2295439723773536e-17 -2.0152132784981046e-17 rpy=0.0 0.0 0.0 -> xyz=-5.78263006557334124e-18 -2.2295439723773536e-17 -2.0152132784981046e-17 rpy=0.0 0 0
- joint joint_iip_middle: origin xyz=0.0004999999999727385 -8.944667923005355e-18 0.04600000000000013 rpy=0.0 0.0 0.0 -> xyz=-0.000499999999972738506 -8.944667923005355e-18 0.04600000000000013 rpy=0.0 0 0
- joint joint_iip_middle_offset: origin xyz=2.1792463666958658e-17 6.938893903907171e-18 -8.326672684688664e-17 rpy=0.0 0.0 0.0 -> xyz=-2.17924636669586576e-17 6.938893903907171e-18 -8.326672684688664e-17 rpy=0.0 0 0
- joint joint_iip_pinky: origin xyz=0.0004999999999844794 -4.138564265705415e-18 0.03300000000000015 rpy=-1.665334536937734e-16 -6.661338147750939e-16 1.1102230246251563e-16 -> xyz=-0.000499999999984479439 -4.138564265705415e-18 0.03300000000000015 rpy=-1.665334536937734e-16 6.66133814775093924e-16 -1.11022302462515629e-16
- joint joint_iip_pinky_offset: origin xyz=1.8619324129843582e-17 3.362886335731112e-17 6.41845325535561e-17 rpy=0.0 0.0 0.0 -> xyz=-1.8619324129843582e-17 3.362886335731112e-17 6.41845325535561e-17 rpy=0.0 0 0
- joint joint_iip_ring: origin xyz=0.0004999999999727302 2.646654142703322e-17 0.045999999999999916 rpy=-6.938893903907228e-17 0.0 -1.1102230246251565e-16 -> xyz=-0.000499999999972730157 2.646654142703322e-17 0.045999999999999916 rpy=-6.938893903907228e-17 0 1.11022302462515654e-16
- joint joint_iip_ring_offset: origin xyz=1.95471717076309e-17 -5.465579791165633e-17 -1.4856164371462412e-17 rpy=0.0 0.0 0.0 -> xyz=-1.95471717076309e-17 -5.465579791165633e-17 -1.4856164371462412e-17 rpy=0.0 0 0
- joint joint_iip_thumb: origin xyz=-2.5364699896779245e-16 5.2599154258198517e-17 -1.0558595790610728e-17 rpy=3.1415926535897927 1.5707963267948948 0.0 -> xyz=2.53646998967792454e-16 5.2599154258198517e-17 -1.0558595790610728e-17 rpy=3.1415926535897927 -1.57079632679489478 0
- joint joint_iip_thumb_offset: origin xyz=-0.0 -0.0 -0.0 rpy=0.0 0.0 0.0 -> xyz=0 -0.0 -0.0 rpy=0.0 0 0
- joint joint_pip_index: origin xyz=9.072004747067653e-17 -2.0636548322369215e-18 9.00862880334811e-18 rpy=7.850462293418878e-17 -1.5707963267948963 0.0 -> xyz=-9.07200474706765258e-17 -2.0636548322369215e-18 9.00862880334811e-18 rpy=7.850462293418878e-17 1.57079632679489634 0
- joint joint_pip_index_offset: origin xyz=-7.643495558336816e-18 -2.0383250328514768e-17 9.34495075168305e-18 rpy=0.0 0.0 0.0 -> xyz=7.64349555833681638e-18 -2.0383250328514768e-17 9.34495075168305e-18 rpy=0.0 0 0
- joint joint_pip_middle: origin xyz=-4.260755233192973e-34 5.7777898331617076e-34 1.301042606982604e-18 rpy=0.0 -1.5707963267948963 0.0 -> xyz=4.26075523319297258e-34 5.7777898331617076e-34 1.301042606982604e-18 rpy=0.0 1.57079632679489634 0
- joint joint_pip_middle_offset: origin xyz=-1.301042606982604e-18 -5.7777898331617076e-34 -7.149650149773824e-34 rpy=0.0 0.0 0.0 -> xyz=1.30104260698260397e-18 -5.7777898331617076e-34 -7.149650149773824e-34 rpy=0.0 0 0
- joint joint_pip_pinky: origin xyz=9.859570060903676e-17 -2.9392458236684397e-17 4.429782895373408e-18 rpy=3.1401849173675513e-16 -1.5707963267948961 0.0 -> xyz=-9.85957006090367584e-17 -2.9392458236684397e-17 4.429782895373408e-18 rpy=3.1401849173675513e-16 1.57079632679489611 0
- joint joint_pip_pinky_offset: origin xyz=7.273901839467707e-19 3.5634470632665727e-17 -4.269871636738011e-17 rpy=0.0 0.0 0.0 -> xyz=-7.27390183946770717e-19 3.5634470632665727e-17 -4.269871636738011e-17 rpy=0.0 0 0
- joint joint_pip_ring: origin xyz=-2.739291165494201e-16 5.658164857459344e-17 -8.813617833534736e-18 rpy=0.0 -1.5707963267948963 0.0 -> xyz=2.73929116549420102e-16 5.658164857459344e-17 -8.813617833534736e-18 rpy=0.0 1.57079632679489634 0
- joint joint_pip_ring_offset: origin xyz=6.29584589194853e-18 -1.1842556896340075e-17 -1.1819659490533676e-16 rpy=0.0 0.0 0.0 -> xyz=-6.29584589194852997e-18 -1.1842556896340075e-17 -1.1819659490533676e-16 rpy=0.0 0 0
- joint joint_pip_thumb: origin xyz=-4.5102810375396984e-17 1.5563939026463913e-16 4.687222832089333e-17 rpy=-1.221730476396032 -4.440892098500626e-16 -9.992007221626409e-16 -> xyz=4.51028103753969845e-17 1.5563939026463913e-16 4.687222832089333e-17 rpy=-1.221730476396032 4.44089209850062616e-16 9.99200722162640886e-16
- joint joint_pip_thumb_offset: origin xyz=-0.03 -0.0 -0.0 rpy=0.0 0.0 0.0 -> xyz=0.0299999999999999989 -0.0 -0.0 rpy=0.0 0 0
- joint middle_ip2middle_fingertip_fixed: origin xyz=-0.009 0.0 0.04 rpy=0.0 0.0 0.0 -> xyz=0.00899999999999999932 0.0 0.04 rpy=0.0 0 0
- joint pinky_ip2pinky_fingertip_fixed: origin xyz=-0.009 0.0 0.04 rpy=0.0 0.0 0.0 -> xyz=0.00899999999999999932 0.0 0.04 rpy=0.0 0 0
- joint ring_ip2ring_fingertip_fixed: origin xyz=-0.009 0.0 0.04 rpy=0.0 0.0 0.0 -> xyz=0.00899999999999999932 0.0 0.04 rpy=0.0 0 0
- joint thumb_dp2thumb_fingertip_fixed: origin xyz=0.0 0.0 0.03 rpy=0.0 0.0 0.0 -> xyz=0 0.0 0.03 rpy=0.0 0 0

Commit message: Fix Orca LEFT URDF mirror: split prismatic/revolute axis rules
The first-pass mirror (3f0d0e6) flipped origins + meshes + renamed sides
but left joint axes unchanged, leaving fingers curling outward instead
of grasping. Three iterations of debugging surfaced the correct rule set:

- Revolute axes follow the YZ-plane pseudovector rule
  (a, b, c) -> (a, -b, -c). Required for fingers and revolute wrist DOFs
  to produce mirrored motion in world frame.
- Prismatic axes deliberately stay world-aligned (1,0,0)/(0,1,0)/(0,0,1).
  retarget_utils.retarget_one_hand short-circuits the IK solver via
  `val += wrist_pos[0/1/2]` on tx/ty/tz joint names, assuming axes
  point world +x/+y/+z. Flipping prismatic axes silently inverts wrist
  placement and colocates the LEFT hand with the RIGHT.
- Joint limits unchanged — under the pseudovector axis flip, positive
  qpos still means flexion on both hands.

Adds verify_chirality.py to encode these rules as a checker so the same
class of bug surfaces as ERROR/WARN instead of silent geometry drift.
Adds render_orca_retarget_viz.py for offline visual confirmation of the
retargeted trajectory.

File: dexmachina/assets/orca_hand/orca_left_6dof.urdf (robot description, URDF)
Before this commit: robot orcahand_v1b_right_6dof, 45 links, 44 joints
Joints:
- joint L_forearm_roll_link_joint: axis 0 0 1 -> 0 0 -1
- joint L_forearm_yaw_link_joint: axis 0 -1 0 -> 0 1 0
- joint joint_abd_index: axis 8.326672684688674e-17 1.1102230246251565e-16 -1.0 -> 8.32667268468867405e-17 -1.11022302462515654e-16 1
- joint joint_abd_middle: axis 4.440892098500626e-16 -4.440892098500626e-16 -0.9999999999999987 -> 4.44089209850062616e-16 4.44089209850062616e-16 0.999999999999998668
- joint joint_abd_pinky: axis -4.996003610813204e-16 -2.7755575615628914e-16 -0.9999999999999987 -> -4.99600361081320443e-16 2.77555756156289135e-16 0.999999999999998668
- joint joint_abd_ring: axis 5.828670879282072e-16 -2.220446049250313e-16 -0.9999999999999996 -> 5.82867087928207184e-16 2.22044604925031308e-16 0.999999999999999556
- joint joint_abd_thumb: axis 0.0 0.0 -1.0 -> 0 0 1
- joint joint_dip_thumb: axis 0.0 -1.0 0.0 -> 0 1 0
- joint joint_iip_index: axis 1.1102230246251565e-16 -0.9999999999999994 3.191891195797325e-16 -> 1.11022302462515654e-16 0.999999999999999445 -3.19189119579732505e-16
- joint joint_iip_middle: axis 6.106226635438361e-16 -0.9999999999999997 -1.035742568734697e-16 -> 6.10622663543836097e-16 0.999999999999999667 1.03574256873469706e-16
- joint joint_iip_pinky: axis 3.885780586188048e-16 -0.9999999999999989 4.718447854656915e-16 -> 3.88578058618804789e-16 0.99999999999999889 -4.7184478546569153e-16
- joint joint_iip_ring: axis -2.220446049250313e-16 -1.0000000000000004 9.298117831235686e-16 -> -2.22044604925031308e-16 1.00000000000000044 -9.29811783123568603e-16
- joint joint_iip_thumb: axis 0.0 -1.0 0.0 -> 0 1 0
- joint joint_pip_index: axis 2.7755575615628914e-16 -1.0000000000000013 3.3306690738754696e-16 -> 2.77555756156289135e-16 1.00000000000000133 -3.33066907387546962e-16
- joint joint_pip_middle: axis 6.106226635438361e-16 -0.9999999999999997 -1.035742568734697e-16 -> 6.10622663543836097e-16 0.999999999999999667 1.03574256873469706e-16
- joint joint_pip_pinky: axis 1.6653345369377348e-16 -0.9999999999999994 -1.1102230246251565e-16 -> 1.66533453693773481e-16 0.999999999999999445 1.11022302462515654e-16
- joint joint_pip_ring: axis -3.3306690738754696e-16 -1.0000000000000007 8.743006318923108e-16 -> -3.33066907387546962e-16 1.00000000000000067 -8.74300631892310776e-16
- joint joint_pip_thumb: axis 0.0 0.34222508701641263 0.9396180020713785 -> 0 -0.342225087016412632 -0.939618002071378466
